File: hardware/Pi Wedge.sch (EAGLE design)
At the start: 15 parts

Commit message: V1.2: Design revisions.
Removing separate 5V and 3.3V connectors.
Integrating 3.3V and 5V in both sides of the DIP-footprint area.
Fixing swapped Tx/Rx on FTDI connector.
Parts:
- removed JP11, JP12: 1x11 Header, SparkFun-Connectors:M111X11_NO_SILK_KIT
- JP2, JP3: value PWR -> M121X12_NO_SILK_KIT; device SparkFun-Connectors:M03PTH -> SparkFun-Connectors:M121X12_NO_SILK_KIT
Connections:
- removed net GPIO17: JP12.2, JP8.GP17
- removed net GPIO18: JP12.3, JP8.GP18#
- removed net GPIO22: JP12.4, JP8.GP22
- removed net GPIO23: JP12.5, JP8.GP23
- removed net GPIO24: JP12.6, JP8.GP24
- removed net GPIO25: JP12.7, JP8.GP25
- removed net GPIO27: JP12.8, JP8.GP27
- removed net GPIO4: JP12.1, JP8.GP4
- new net GP17: JP3.4, JP8.GP17
- new net GP18: JP3.5, JP8.GP18#
- new net GP22: JP3.6, JP8.GP22
- new net GP23: JP3.7, JP8.GP23
- new net GP24: JP3.8, JP8.GP24
- new net GP25: JP3.9, JP8.GP25
- new net GP27: JP3.10, JP8.GP27
- new net GP4: JP2.4, JP8.GP4
- net 3.3V: now also JP2.2, JP3.2; no longer JP11.1, JP2.1, JP3.1
- net 5V: no longer JP11.2
- net CE0: now also JP2.10; no longer JP11.8
- net CE1: now also JP2.11; no longer JP11.9
- net GND: now also JP2.1, JP2.12, JP3.1; no longer JP11.10, JP11.11, JP12.11, JP2.2, JP3.2
- net MISO: now also JP2.8; no longer JP11.6
- net MOSI: now also JP2.9; no longer JP11.7
- net RXI: now also JP2.6, JP4.RXI; no longer JP11.4, JP4.TXO
- net SCL: now also JP3.12; no longer JP12.10
- net SCLK: now also JP2.7; no longer JP11.5
- net SDA: now also JP3.11; no longer JP12.9
- net TXO: now also JP2.5, JP4.TXO; no longer JP11.3, JP4.RXI
Other:
- note added: "V12"
- note removed: "V10"

Commit message: Swapping in new breadboard reference symbol.
No changes to the board itself.
Parts:
- added U$2: BREADBOARD_PATTERN, SparkFun-Aesthetics:BREADBOARD_PATTERN
Changed lines of the file:
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@@
 <part name="SUPPLY5" library="SparkFun-Aesthetics" deviceset="3.3V" device=""/>
 <part name="SUPPLY6" library="SparkFun-Aesthetics" deviceset="5V" device=""/>
+<part name="U$2" library="SparkFun-Aesthetics" deviceset="BREADBOARD_PATTERN" device=""/>
 </parts>
 <sheets>
@@
 <instance part="SUPPLY5" gate="G$1" x="182.88" y="134.62"/>
 <instance part="SUPPLY6" gate="G$1" x="177.8" y="134.62"/>
+<instance part="U$2" gate="G$1" x="225.298" y="5.842"/>
 </instances>
 <busses>
